File: robot_arm_board-double_sided/robot_arm.kicad_pcb (KiCad board)
At the start: 2 copper layers, 94.9 x 71.1 mm, 33 parts, among them J1 microstepping, J10 microstepping, J11 microstepping, J12 microstepping, J13 microstepping, J14 Screw_Terminal_01x02, J15 Screw_Terminal_01x02, J16 I2C, J18 fan, J19 SW_PINS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

Commit message: atualizações no modelo
Routing:
- net Net-(A2-DIR): track 23.3 -> 21.2 mm
- net Net-(A2-STEP): track 27.9 -> 25.8 mm
- added copper zone on B.Cu, net GND
